File: IoT_Dimmer.kicad_sch (KiCad schematic)
At the start: 52 parts, among them J1 Wago_2059-302998-403:CONN2_20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, J2 Screw_Terminal_01x02, J3 Conn_01x06_Pin, SW1 EVE-SBBFE516B, U1 MOC3021S, U2 VOS628AT, U3 ESP32-C6FH4, Y2 Crystal_GND24

Commit message: CPU_STAND
Parts:
- C3, C4: footprint Capacitor_SMD:C_0603_1608Metric -> Capacitor_SMD:C_0402_1005Metric
- L1: footprint Inductor_SMD:L_0805_2012Metric -> Inductor_SMD:L_0402_1005Metric
- L2: footprint Inductor_SMD:L_0805_2012Metric -> Inductor_SMD:L_0603_1608Metric
Connections:
- net xtal_n renamed XTAL_N
- net xtal_p renamed XTAL_P
Changed lines of the file:
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@@
 		)
 	)
-	(label "xtal_n"
+	(label "XTAL_N"
 		(at 67.31 114.3 180)
 		(effects
@@
 		)
 	)
-	(label "xtal_p"
+	(label "XTAL_P"
 		(at 67.31 127 180)
 		(effects
@@
 			)
 		)
-		(property "Footprint" "Inductor_SMD:L_0805_2012Metric"
+		(property "Footprint" "Inductor_SMD:L_0603_1608Metric"
 			(at 74.93 34.29 0)
 			(effects
@@
 			)
 		)
-		(property "Footprint" "Inductor_SMD:L_0805_2012Metric"
+		(property "Footprint" "Inductor_SMD:L_0402_1005Metric"
 			(at 43.18 57.15 0)
 			(effects
@@
 			)
 		)
-		(property "Footprint" "Capacitor_SMD:C_0603_1608Metric"
+		(property "Footprint" "Capacitor_SMD:C_0402_1005Metric"
 			(at 50.4952 67.31 0)
 			(effects
@@
 			)
 		)
-		(property "Footprint" "Capacitor_SMD:C_0603_1608Metric"
+		(property "Footprint" "Capacitor_SMD:C_0402_1005Metric"
 			(at 36.5252 67.31 0)
 			(effects

Commit message: pcb
Parts:
- renumbered C7 to C1, C11 to C10, C14 to C11, C16 to C12, C17 to C13, C10 to C14, C9 to C15, C21 to C16, C19 to C17, C1 to C19, C4 to C2, C2 to C21, C5 to C3, C3 to C4, C6 to C5, C8 to C6, C13 to C7, C12 to C8, C15 to C9, J3 to J1, J1 to J3, R6 to R1, R4 to R10, R5 to R11, R1 to R12, R2 to R13, R3 to R14, R7 to R2, R8 to R3, R9 to R4, R11 to R5, R10 to R6, R12 to R7, R13 to R8, R14 to R9, TP2 to TP1, TP1 to TP2, U3 to U1, U1 to U3, Y2 to Y1
